Commit message: raggiunge 4 way points e quindi i 4 punti del piano

File: urdf/robot4.xacro (robot description, xacro)
@@ -1,5 +1,5 @@
 <?xml version="1.0"?>
 <robot xmlns:xacro="http://www.ros.org/wiki/xacro" name="robot4_xacro">
-<xacro:include filename="$(find robot_urdf)/urdf/robot4.gazebo"/>
+<xacro:include filename="$(find assignment2_exprob)/urdf/robot4.gazebo"/>
 	<xacro:property name="length_wheel" value="0.04" />
 	<xacro:property name="radius_wheel" value="0.1" />
@@ -175,3 +175,31 @@
 	</actuator>
    </transmission>
+ <link name="hokuyo_link">
+	    <collision>
+	      <origin xyz="0 0 0.025" rpy="0 0 0"/>
+	      <geometry>
+		<box size="0.05 0.05 0.05"/>
+	      </geometry>
+	    </collision>
+	    <visual>
+	      <origin xyz="0 0 0.025" rpy="0 0 0"/>
+	      <geometry>
+		<box size="0.05 0.05 0.05"/>
+	      </geometry>
+	      <material name="red">
+		<color rgba="1 0 0 1"/>
+	      </material>
+	    </visual>
+	    <inertial>
+	      <mass value="1e-5" />
+	      <origin xyz="0 0 0" rpy="0 0 0"/>
+	      <inertia ixx="1e-6" ixy="0" ixz="0" iyy="1e-6" iyz="0" izz="1e-6" />
+	    </inertial>
+ 	 </link>
+ 	 <joint name="hokuyo_joint" type="fixed">
+	    <axis xyz="0 1 0" />
+	    <origin xyz="0.26 0 0.01" rpy="0 0 0"/>
+	    <parent link="link_chassis"/>
+	    <child link="hokuyo_link"/>
+	 </joint>
 </robot>

Commit message: Finito da ridefinire

File: urdf/robot4.xacro (robot description, xacro)
@@ -115,15 +115,15 @@
     <joint_properties damping="1.0" friction="1.0"/>
   </joint>
-    <link name="support_camera_link">
-	    <collision>
-	      <origin xyz="0 0 0.1" rpy="0 0 0"/>
-	      <geometry>
-		<box size="0.05 0.05 0.2"/>
-	      </geometry>
-	    </collision>
-	    <visual>
-	      <origin xyz="0 0 0.1" rpy="0 0 0"/>
-	      <geometry>
-		<box size="0.05 0.05 0.2"/>
+    <link name="support_camera_link_0">
+	    <collision>
+	      <origin xyz="0 0 0" rpy="0 0 0"/>
+	      <geometry>
+		<box size="0.05 0.05 0.18"/>
+	      </geometry>
+	    </collision>
+	    <visual>
+	      <origin xyz="0 0 0.05" rpy="0 0 0"/>
+	      <geometry>
+		<box size="0.05 0.05 0.18"/>
 	      </geometry>
 	      <material name="blue"/>
@@ -131,25 +131,53 @@
 	    <inertial>
 	      <mass value="1e-5" />
-	      <origin xyz="0 0 0.1" rpy="0 0 0"/>
+	      <origin xyz="0 0 0.0" rpy="0 0 0"/>
 	      <inertia ixx="1e-6" ixy="0" ixz="0" iyy="1e-6" iyz="0" izz="1e-6" />
-	    </inertial>
-  </link>
-  <joint name="support_camera_joint" type="fixed">
+	    </inertial> 02
+  </link>
+  <joint name="support_camera_joint_0" type="fixed">
 	    <axis xyz="0 0 1" />
-	    <origin xyz="0 0 0.002" rpy="0 0 0"/>
+	    <origin xyz="0 0 0.01" rpy="0 0 0"/>
+	    <child link="support_camera_link_0"/>
+	    <parent link="link_chassis"/>
+	 </joint>
+  <link name="support_camera_link">
+	    <collision>
+	      <origin xyz="0 0 0.07" rpy="0 0 0"/>
+	      <geometry>
+		<box size="0.2 0.05 0.05"/>
+	      </geometry>
+	    </collision>
+	    <visual>
+	      <origin xyz="0.0 0 0.07" rpy="0 0 0"/>
+	      <geometry>
+		<box size="0.2 0.05 0.05"/>
+	      </geometry>
+	      <material name="blue"/>
+	    </visual>
+	    <inertial>
+	      <mass value="1e-5" />
+	      <origin xyz="0 0 0" rpy="0 0 0"/>
+	      <inertia ixx="1e-6" ixy="0" ixz="0" iyy="1e-6" iyz="0" izz="1e-6" />
+	    </inertial> 02
+  </link>
+  <joint name="support_camera_joint" type="continuous">
+	    <axis xyz="0 0 1" />
+	    <origin xyz="0.075 0 0.09" rpy="0 0 0"/>
+	    <dynamics damping="0.1"/>
+        <limit effort="10000" velocity="100" />
 	    <child link="support_camera_link"/>
-	    <parent link="link_chassis"/>
+	    <parent link="support_camera_link_0"/>
 	 </joint>
   <link name="camera_link">
 	    <collision>
-	      <origin xyz="0.1 0 0.00" rpy="0 0 0"/>
-	      <geometry>
-		<box size="0.05 0.05 0.05"/>
-	      </geometry>
-	    </collision>
-	    <visual>
-	      <origin xyz="0.0 0 0.05" rpy="0 0 0"/>
-	      <geometry>
-		<box size="0.1 0.1 0.05"/>
+	      <origin xyz="0.05 0.05 0.05" rpy="0 0 0"/>
+	      <geometry>
+		<box size="0.05 0.05 0.05"/>
+	      </geometry>
+	    </collision>
+	    <visual>
+	      <origin xyz="0.00 0 0.00" rpy="0 0 0"/>
+	      <geometry>
+		<box size="0.05 0.05 0.05"/>
 	      </geometry>
 	      <material name="red"/>
@@ -157,9 +185,7 @@
 	   <xacro:default_inertial mass="0.02"/>
   </link>
-  <joint name="camera_joint" type="continuous">
-	    <axis xyz="0 0 1" />
-        <origin xyz="0.0 0.0 0.175" rpy="0 0 0"/>
-        <dynamics damping="0.1"/>
-        <limit effort="10000" velocity="100" />
+  <joint name="camera_joint" type="fixed">
+	    <axis xyz="0 1 0" />
+        <origin xyz="0.125 0.0 0.07" rpy="0 0 0"/>
 	    <child link="camera_link"/>
 	    <parent link="support_camera_link"/>
@@ -167,5 +193,5 @@
   <transmission name="camera_joint_trans">
 	<type>transmission_interface/SimpleTransmission</type>
-	<joint name="camera_joint">
+	<joint name="support_camera_joint">
 		<hardwareInterface>hardware_interface/VelocityJointInterface</hardwareInterface>
 	</joint>
